File: sensor.kicad_sch (KiCad schematic)
At the start: 4 parts, among them U2 SLSS49E-3

Commit message: Setup Base Layout
Parts:
- renumbered C22 to C7, C27 to C8, R4 to R1, U2 to SW1

Commit message: Routed a lot of the pcb, additionally fixed issues with wrong layout
Parts:
- renumbered C7 to C11, C8 to C12, R1 to R4, SW1 to SW2
